File: toy_car_motor_driver.kicad_sch (KiCad schematic)
At the start: 15 parts, among them J1 Conn_01x06_Pin, J3 Conn_01x02_Pin, J4 Screw_Terminal_01x02, J5 Screw_Terminal_01x02, J6 Screw_Terminal_01x02, SW1 SW_DIP_x04, U1 L293D

Commit message: made further changes
Connections:
- net 9V_i: now also SW1.1; no longer SW1.2
- net GND_i: now also SW1.2; no longer SW1.1
Other:
- moved on the sheet: J6
Changed lines of the file:
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@@
     (stroke (width 0) (type default))
   )
-  (wire (pts (xy 58.42 39.37) (xy 54.61 39.37))
+  (wire (pts (xy 44.45 39.37) (xy 58.42 39.37))
     (stroke (width 0) (type default))
   )
@@
     (stroke (width 0) (type default))
   )
-  (wire (pts (xy 54.61 36.83) (xy 62.23 36.83))
+  (wire (pts (xy 44.45 36.83) (xy 62.23 36.83))
     (stroke (width 0) (type default))
   )
@@
     (effects (font (size 1.27 1.27)) (justify right bottom))
   )
-  (label "GND_i" (at 54.61 36.83 0) (fields_autoplaced)
+  (label "GND_i" (at 53.34 39.37 0) (fields_autoplaced)
     (effects (font (size 1.27 1.27)) (justify left bottom))
   )
@@
     (effects (font (size 1.27 1.27)) (justify right bottom))
   )
-  (label "9V_i" (at 54.61 39.37 0) (fields_autoplaced)
+  (label "9V_i" (at 54.61 36.83 0) (fields_autoplaced)
     (effects (font (size 1.27 1.27)) (justify left bottom))
   )
@@
     )
   )
-  (symbol (lib_id "Connector:Screw_Terminal_01x02") (at 49.53 39.37 180) (unit 1)
-    (in_bom yes) (on_board yes) (dnp no) (fields_autoplaced)
-    (property "Reference" "J6" (at 49.53 30.48 0)
-      (effects (font (size 1.27 1.27)))
-    )
-    (property "Value" "Screw_Terminal_01x02" (at 49.53 33.02 0)
-      (effects (font (size 1.27 1.27)))
-    )
-    (property "Footprint" "Connector:JWT_A3963_1x02_P3.96mm_Vertical" (at 49.53 39.37 0)
-      (effects (font (size 1.27 1.27)) hide)
-    )
-    (property "Datasheet" "~" (at 49.53 39.37 0)
-      (effects (font (size 1.27 1.27)) hide)
-    )
+  (symbol (lib_id "Connector:Screw_Terminal_01x02") (at 49.53 36.83 0) (unit 1)
+    (in_bom yes) (on_board yes) (dnp no) (fields_autoplaced)
+    (property "Reference" "J6" (at 52.07 36.83 0)
+      (effects (font (size 1.27 1.27)) (justify left))
+    )
+    (property "Value" "Screw_Terminal_01x02" (at 52.07 39.37 0)
+      (effects (font (size 1.27 1.27)) (justify left))
+    )
+    (property "Footprint" "Connector:JWT_A3963_1x02_P3.96mm_Vertical" (at 49.53 36.83 0)
+      (effects (font (size 1.27 1.27)) hide)
+    )
+    (property "Datasheet" "~" (at 49.53 36.83 0)
+      (effects (font (size 1.27 1.27)) hide)
+    )

Commit message: Updated pcb
Parts:
- removed SW1: SW_DIP_x04, Package_DIP:DIP-8_W7.62mm, symbol Switch:SW_DIP_x04
Connections:
- net 5V_i is gone; now on net 5V: J3.1 (Pin_1)
- net 9V_i is gone; now on net 9V: J6.1 (Pin_1)
- net GND_i is gone; now on net GND: J3.2 (Pin_2), J6.2 (Pin_2)
Other:
- moved on the sheet: D1, J6, R1
